File: hardware/duodrive.kicad_pcb (KiCad board)
At the start: 2 copper layers, 49 x 75 mm, 113 parts, among them J2 Conn_02x08_Odd_Even, J3 SWD, J4 CAN_IN, J5 CAN_OUT, J6 POWER, J7 ENCODER1, J8 ENCODER2, Q1 AOD4184, Q2 AOD4184, Q3 AOD4184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

Commit message: layout and component changes
Parts:
- removed C28: 22uF, Capacitor_SMD:C_1206_3216Metric
- removed D2, D21, D3: LED_Small, LED_SMD:LED_0603_1608Metric
- added D4: LED_KRGB, LED_SMD:LED_RGB_1210, F.Cu at (114.5, 86.9)
- added JP1: Jumper_2_Open, Jumper:SolderJumper-2_P1.3mm_Open_RoundedPad1.0x1.5mm, B.Cu at (134.4, 103.6)
- added R23: 120R, Resistor_SMD:R_0603_1608Metric, F.Cu at (133.8, 106.4)
- C18, C20, C27: value 22uF -> 10uF
- C25: value 33nF -> 100nF
- C29: value 10uF -> 22uF
- J4, J5: footprint Connector_JST:JST_SH_SM04B-SRSS-TB_1x04-1MP_P1.00mm_Horizontal -> Connector_Molex:Molex_PicoBlade_53261-0471_1x04-1MP_P1.25mm_Horizontal
- JP2: footprint Connector_PinHeader_2.54mm:PinHeader_1x03_P2.54mm_Vertical -> Jumper:SolderJumper-3_P1.3mm_Open_RoundedPad1.0x1.5mm; moved to B.Cu
- Q1, Q2, Q3, Q4, Q5, Q7: value AOD4184 -> DON50N04; footprint Package_TO_SOT_SMD:TO-252-2 -> Package_DFN_QFN:PQFN-8-EP_6x5mm_P1.27mm_Generic
- Q6, Q8: value AOD4184 -> NMOS-8PINS; footprint Package_TO_SOT_SMD:TO-252-2 -> Package_DFN_QFN:PQFN-8-EP_6x5mm_P1.27mm_Generic
- R12: value 10K -> 56K
- R7: value 10K -> 470K
- TP1, TP2: footprint TestPoint:TestPoint_THTPad_D1.0mm_Drill0.5mm -> TestPoint:TestPoint_Pad_D1.0mm
- U2, U5, U6, U7: value IR2011 -> UCC27211
- moved R9 26.6 mm to (110.0, 86.1)
- moved D1 24.2 mm to (92.4, 115.0), turned to 90 degrees
- moved R1 21.7 mm to (92.4, 112.0), turned to -90 degrees
- moved R10 20.1 mm to (110.0, 87.7), turned to 0 degrees
- moved R3 11.8 mm to (118.4, 86.9)
- moved C18 7.61 mm to (128.9, 97.7), turned to -90 degrees
- moved C41 6.30 mm to (117.8, 96.1), turned to 180 degrees
- moved J4 6.21 mm to (136.1, 100.5)
- moved R12 6.11 mm to (130.9, 102.3)
- moved R7 6.11 mm to (130.9, 100.8)
- moved L1 6.10 mm to (125.5, 97.7)
- moved U8 5.95 mm to (128.1, 101.4)
- moved C25 5.65 mm to (125.2, 102.3)
- moved C6 5.65 mm to (125.2, 100.8)
- moved C27 5.42 mm to (131.2, 97.7), turned to -90 degrees
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Connections:
- D1 pad 1: GND -> GNDS
- D20 pad 1: Net-(D20-K) -> GNDS
- D20 pad 2: +3.3V -> Net-(D20-A)
- Q1 pad 1: Net-(D6-A) -> MOTOR_OUT_1
- Q1 pad 2: VDC -> MOTOR_OUT_1
- Q2 pad 1: Net-(D7-A) -> GND
- Q2 pad 2: MOTOR_OUT_1 -> GND
- Q3 pad 1: Net-(D10-A) -> MOTOR_OUT_2
- Q3 pad 2: VDC -> MOTOR_OUT_2
- Q4 pad 1: Net-(D11-A) -> GND
- Q4 pad 2: MOTOR_OUT_2 -> GND
- Q5 pad 1: Net-(D13-A) -> MOTOR_OUT_3
- Q5 pad 2: VDC -> MOTOR_OUT_3
- Q6 pad 1: Net-(D14-A) -> GND
- Q6 pad 2: MOTOR_OUT_3 -> GND
- Q7 pad 1: Net-(D15-A) -> MOTOR_OUT_4
- Q7 pad 2: VDC -> MOTOR_OUT_4
- Q8 pad 1: Net-(D16-A) -> GND
- Q8 pad 2: MOTOR_OUT_4 -> GND
- R3 pad 1: LED2 -> LED4
- R8 pad 1: Net-(D20-K) -> +3.3V
- R8 pad 2: GNDS -> Net-(D20-A)
- R9 pad 1: LED4 -> LED2
- U4 pad 14: unconnected-(U4-PA2-Pad14) -> LED1
- U4 pad 59: LED1 -> unconnected-(U4-PB6-Pad59)
Routing:
- net LED3: track 31.6 -> 13.0 mm, vias 4 -> 2
- net LED4: track 35.6 -> 21.1 mm
- net +10V: track 80.5 -> 87.6 mm
- net VBUS: track 18.1 -> 11.1 mm
- net LED2: track 10.3 -> 15.2 mm
- net Net-(D10-A): track 16.9 -> 20.8 mm, vias 0 -> 2
- net +3.3V: track 109.2 -> 105.5 mm, vias 2 -> 1
- net Net-(D6-A): track 17.5 -> 21.2 mm, vias 0 -> 2
- net Net-(D13-A): track 17.2 -> 20.7 mm, vias 0 -> 2
- net +5V: track 76.6 -> 73.4 mm
- net VDC: track 45.5 -> 42.4 mm
- net Net-(D15-A): track 17.3 -> 20.2 mm, vias 0 -> 2
- net CAN_L: track 14.0 -> 16.8 mm, vias 2 -> 0
- net MOTOR_OUT_1: track 15.7 -> 18.1 mm, vias 112 -> 117
- net Net-(U8-RT): track 4.70 -> 2.69 mm
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Other:
- board text added: "+"
- board text added: "-"
- board text added: "V2.2"
- board text removed: "V2.1"
