File: hardware/duodrive.kicad_sch (KiCad schematic)
At the start: 112 parts, among them J2 Conn_02x08_Odd_Even, J3 SWD, J4 CAN_IN, J5 CAN_OUT, J6 POWER, J7 ENCODER1, J8 ENCODER2, Q1 AOD4184, Q2 AOD4184, Q3 AOD4184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

Commit message: polishing
Other:
- moved on the sheet: C1, C11, C13, C14, C15, C16, C17, C19, C2, C21, C22, C3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

Commit message: polishing
Parts:
- R4: value 11.8K -> 115K
- R6: value 1K -> 10K
Connections:
- net CANSET: no longer names the net of U4.34 (PB12)
Changed lines of the file:
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@@
 	(wire
 		(pts
-			(xy 60.96 173.99) (xy 60.96 175.26)
-		)
-		(stroke
-			(width 0)
-			(type default)
-		)
-	)
-	(wire
-		(pts
 			(xy 353.06 60.96) (xy 353.06 69.85)
 		)
@@
 	(global_label "Reset"
 		(shape input)
-		(at 60.96 175.26 180)
+		(at 60.96 173.99 180)
 		(fields_autoplaced yes)
 		(effects
@@
 		)
 		(property "Intersheetrefs" "${INTERSHEET_REFS}"
-			(at 52.7738 175.26 0)
+			(at 52.7738 173.99 0)
 			(effects
 				(font
@@
 		)
 	)
-	(global_label "CANSET"
-		(shape input)
-		(at 96.52 242.57 0)
-		(fields_autoplaced yes)
-		(effects
-			(font
-				(size 1.27 1.27)
-			)
-			(justify left)
-		)
-		(property "Intersheetrefs" "${INTERSHEET_REFS}"
-			(at 106.5204 242.57 0)
-			(effects
-				(font
-					(size 1.27 1.27)
-				)
-				(justify left)
-				(hide yes)
-			)
-		)
-	)
 	(global_label "PWM1A"
 		(shape input)
@@
 			)
 		)
-		(property "Value" "1K"
+		(property "Value" "10K"
 			(at 139.7 67.31 90)
 			(effects
@@
 			)
 		)
-		(property "Value" "11.8K"
+		(property "Value" "115K"
 			(at 139.7 59.69 90)
 			(effects
